File: MCU DATALOGGER.kicad_pcb (KiCad board)
At the start: 2 copper layers, 30 parts, among them J1 Conn_01x04_Pin, J2 Conn_01x04_Pin, J3 Conn_01x09_Pin, J4 Conn_02x03_Odd_Even, U1 24LC1025, U2 24LC1025, U3 ATMEGA328P-AU, U4 DS1337S_, Y1 16MHz, Y2 32.768 KHz

Commit message: done the placing
Parts:
- removed H5: MountingHole, MountingHole:MountingHole_2.1mm
- moved J3 104.4 mm to (66.7, 98.0), turned to 90 degrees
- moved BT1 98.5 mm to (63.5, 77.8)
- moved Y2 94.7 mm to (63.8, 87.2), turned to 90 degrees
- moved J2 88.9 mm to (92.0, 98.0), turned to 90 degrees
- moved C3 83.3 mm to (73.8, 92.5)
- moved C4 79.6 mm to (78.2, 83.8), turned to 90 degrees
- moved C2 76.9 mm to (80.2, 83.8), turned to 90 degrees
- moved U4 76.2 mm to (72.2, 88.5)
- moved J1 76.1 mm to (99.5, 94.0), turned to -90 degrees
- moved J4 75.9 mm to (97.2, 77.0)
- moved Y1 75.4 mm to (84.0, 87.8), turned to 180 degrees
- moved U2 75.2 mm to (72.5, 80.5)
- moved U1 75.2 mm to (72.6, 73.8)
- moved H4 73.0 mm to (62.5, 97.2)
- moved H1 72.8 mm to (62.5, 71.8)
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Other:
- board outline added: 47.5 x 30.5 mm

Commit message: Done with layout
Parts:
- moved J2 1.25 mm to (92.0, 96.8)
- moved J3 1.25 mm to (66.7, 96.8)
- moved J1 1.00 mm to (99.5, 93.0)
Routing:
- net /VCC: track 0.00 -> 128.1 mm, vias 0 -> 5
- net GND: track 0.00 -> 85.1 mm, vias 0 -> 11
- net /SCK: track 0.00 -> 68.1 mm, vias 0 -> 8
- net /SDA: track 0.00 -> 57.2 mm, vias 0 -> 5
- net Net-(BT1-+): track 0.00 -> 55.4 mm, vias 0 -> 7
- net /D3: track 0.00 -> 47.2 mm, vias 0 -> 2
- net /D2: track 0.00 -> 46.2 mm
- net /D4: track 0.00 -> 38.7 mm, vias 0 -> 2
- net /TX: track 0.00 -> 34.5 mm, vias 0 -> 2
- net /RX: track 0.00 -> 32.0 mm, vias 0 -> 2
- net Net-(U3-PB7): track 0.00 -> 23.6 mm, vias 0 -> 2
- net /RESET: track 0.00 -> 22.0 mm, vias 0 -> 1
- net /D6: track 0.00 -> 19.2 mm, vias 0 -> 2
- net /D5: track 0.00 -> 18.9 mm, vias 0 -> 3
- net Net-(U3-AREF): track 0.00 -> 18.1 mm, vias 0 -> 2
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- added copper zone on B.Cu, net GND

Commit message: Done
Connections:
- BT1 pad 1: Net-(BT1-+) -> /VCC
- C5 pad 1: Net-(BT1-+) -> /VCC
- D1 pad 2: Net-(BT1-+) -> /VCC
- U3 pad 18: Net-(BT1-+) -> /VCC
- U3 pad 6: Net-(BT1-+) -> /VCC
Routing:
- net Net-(BT1-+): track 55.4 -> 0.00 mm, vias 7 -> 0
- net /VCC: track 128.1 -> 177.1 mm, vias 5 -> 9
- net GND: track 85.1 -> 86.5 mm, vias 11 -> 12
Other:
- board text added: "GND"
- board text added: "RX"
- board text added: "SCK"
- board text added: "SDA"
- board text added: "TX"
- board text added: "VCC"
